File: FADETUBE_MIDI/FADETUBE_MIDI.kicad_pcb (KiCad board)
At the start: 2 copper layers, 7 parts, among them J1 B8B-XH-A, J2 B8B-XH-A, J3 B8B-PH-K-S, J4 B8B-PH-K-S, U1 Sparkfun_Pro_Micro

Commit message: updates
Parts:
- removed J1, J2: B8B-XH-A, FADETUBE_LIBRARY:JST_B8B-XH-A
- added G***: LOGO, FADETUBE_LIBRARY:onda-audio-logo, F.Cu at (176.5, 150.0)
- added G***: LOGO, FADETUBE_LIBRARY:fadetube-logo, F.Cu at (166.0, 150.0)
- moved J1_DECK_A1 10.1 mm to (129.0, 142.4)
- moved J2_DECK_B1 9.45 mm to (171.0, 142.5)
- renumbered U1 to ArduinoProMicroATmega32U4USB-C1, R1 to FADER1, J3 to J1_DECK_A1, J4 to J2_DECK_B1, S1 to ROTARY_ENCODER_BTN1
Connections:
- ArduinoProMicroATmega32U4USB-C1 pad 10: unconnected-(U1-D7-Pad10) -> Net-(ArduinoProMicroATmega32U4USB-C1-D7)
- ArduinoProMicroATmega32U4USB-C1 pad 11: unconnected-(U1-D8/A8-Pad11) -> Net-(ArduinoProMicroATmega32U4USB-C1-D8/A8)
- ArduinoProMicroATmega32U4USB-C1 pad 12: unconnected-(U1-~D9/A9-Pad12) -> Net-(ArduinoProMicroATmega32U4USB-C1-~D9/A9)
- ArduinoProMicroATmega32U4USB-C1 pad 13: unconnected-(U1-~D10/A10-Pad13) -> Net-(ArduinoProMicroATmega32U4USB-C1-~D10/A10)
- ArduinoProMicroATmega32U4USB-C1 pad 14: unconnected-(U1-D16-Pad14) -> Net-(ArduinoProMicroATmega32U4USB-C1-D16)
- ArduinoProMicroATmega32U4USB-C1 pad 15: unconnected-(U1-D14-Pad15) -> Net-(ArduinoProMicroATmega32U4USB-C1-D14)
- ArduinoProMicroATmega32U4USB-C1 pad 21: unconnected-(U1-VCC-Pad21) -> Net-(ArduinoProMicroATmega32U4USB-C1-VCC)
- ArduinoProMicroATmega32U4USB-C1 pad 3: unconnected-(U1-GND-Pad3) -> GND
- ArduinoProMicroATmega32U4USB-C1 pad 4: Net-(S1-Pad2) -> GND
- ArduinoProMicroATmega32U4USB-C1 pad 7: unconnected-(U1-D4/A6-Pad7) -> Net-(ArduinoProMicroATmega32U4USB-C1-D4/A6)
- ArduinoProMicroATmega32U4USB-C1 pad 8: unconnected-(U1-~D5-Pad8) -> Net-(ArduinoProMicroATmega32U4USB-C1-~D5)
- ArduinoProMicroATmega32U4USB-C1 pad 9: unconnected-(U1-~D6/A7-Pad9) -> Net-(ArduinoProMicroATmega32U4USB-C1-~D6/A7)
- FADER1 pad 3: VCC -> Net-(ArduinoProMicroATmega32U4USB-C1-VCC)
- J1_DECK_A1 pad 1: unconnected-(J3-Pad1) -> Net-(ArduinoProMicroATmega32U4USB-C1-~D5)
- J1_DECK_A1 pad 2: unconnected-(J3-Pad2) -> Net-(ArduinoProMicroATmega32U4USB-C1-~D9/A9)
- J1_DECK_A1 pad 3: unconnected-(J3-Pad3) -> GND
- J1_DECK_A1 pad 4: unconnected-(J3-Pad4) -> GND
- J1_DECK_A1 pad 5: unconnected-(J3-Pad5) -> Net-(ArduinoProMicroATmega32U4USB-C1-D7)
- J1_DECK_A1 pad 6: unconnected-(J3-Pad6) -> Net-(ArduinoProMicroATmega32U4USB-C1-D16)
- J1_DECK_A1 pad 7: unconnected-(J3-Pad7) -> GND
- J1_DECK_A1 pad 8: unconnected-(J3-Pad8) -> GND
- J2_DECK_B1 pad 1: unconnected-(J4-Pad1) -> Net-(ArduinoProMicroATmega32U4USB-C1-~D6/A7)
- J2_DECK_B1 pad 2: unconnected-(J4-Pad2) -> Net-(ArduinoProMicroATmega32U4USB-C1-~D10/A10)
- J2_DECK_B1 pad 3: unconnected-(J4-Pad3) -> GND
- J2_DECK_B1 pad 4: unconnected-(J4-Pad4) -> GND
- J2_DECK_B1 pad 5: unconnected-(J4-Pad5) -> Net-(ArduinoProMicroATmega32U4USB-C1-D8/A8)
- J2_DECK_B1 pad 6: unconnected-(J4-Pad6) -> Net-(ArduinoProMicroATmega32U4USB-C1-D14)
- J2_DECK_B1 pad 7: unconnected-(J4-Pad7) -> GND
- J2_DECK_B1 pad 8: unconnected-(J4-Pad8) -> GND
- ROTARY_ENCODER_BTN1 pad 2: Net-(S1-Pad2) -> Net-(ArduinoProMicroATmega32U4USB-C1-D4/A6)
Routing:
- net GND: track 0.00 -> 152.1 mm
- net Net-(ArduinoProMicroATmega32U4USB-C1-VCC): track 0.00 -> 88.0 mm, vias 0 -> 1
- net Net-(ArduinoProMicroATmega32U4USB-C1-D14): track 0.00 -> 76.5 mm, vias 0 -> 1
- net Net-(ArduinoProMicroATmega32U4USB-C1-D8/A8): track 0.00 -> 74.1 mm, vias 0 -> 1
- net Net-(ArduinoProMicroATmega32U4USB-C1-~D6/A7): track 0.00 -> 71.5 mm, vias 0 -> 1
- net Net-(FADER1-SHIELD-PadSH1): track 0.00 -> 68.2 mm
- net Net-(ArduinoProMicroATmega32U4USB-C1-~D10/A10): track 0.00 -> 64.5 mm, vias 0 -> 1
- net Net-(ArduinoProMicroATmega32U4USB-C1-~D5): track 0.00 -> 45.8 mm, vias 0 -> 1
- net Net-(ArduinoProMicroATmega32U4USB-C1-D7): track 0.00 -> 36.2 mm
- net Net-(ArduinoProMicroATmega32U4USB-C1-~D9/A9): track 0.00 -> 35.8 mm, vias 0 -> 1
- net Net-(ArduinoProMicroATmega32U4USB-C1-D4/A6): track 0.00 -> 34.8 mm, vias 0 -> 1
- net Net-(ArduinoProMicroATmega32U4USB-C1-D16): track 0.00 -> 32.4 mm
- net Net-(ArduinoProMicroATmega32U4USB-C1-D18/A0): track 0.00 -> 25.8 mm
- net Net-(ArduinoProMicroATmega32U4USB-C1-D2): track 0.00 -> 18.9 mm
- net Net-(ROTARY_ENCODER_BTN1-SHIELD-PadSH1): track 0.00 -> 18.0 mm
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Other:
- board outline added: 70 x 70 mm
- board text added: "FADETUBE DJ MIDI CONTROLLER v01.00 MARIO D. QUIROZ / ONDAAUDIO.MX"

Commit message: test smd
Parts:
- added R1_PLAY_A1: 1k, Resistor_SMD:R_0603_1608Metric, F.Cu at (141.5, 142.0)
- added R_LOAD_A1: 1k, Resistor_SMD:R_0603_1608Metric, F.Cu at (147.5, 142.0)
- added R_LOAD_B1: 1k, Resistor_SMD:R_0603_1608Metric, F.Cu at (153.5, 141.8)
- added R_PLAY_B1: 1k, Resistor_SMD:R_0603_1608Metric, F.Cu at (158.0, 142.0)
- renumbered G*** to FADETUBE-LOGO, G*** to ONDAAUDIO-LOGO
Connections:
- J1_DECK_A1 pad 2: Net-(ArduinoProMicroATmega32U4USB-C1-~D9/A9) -> Net-(SW_PLAY_A1-A)
- J1_DECK_A1 pad 6: Net-(ArduinoProMicroATmega32U4USB-C1-D16) -> Net-(SW_LOAD_A1-A)
- J2_DECK_B1 pad 2: Net-(ArduinoProMicroATmega32U4USB-C1-~D10/A10) -> Net-(SW_PLAY_B1-A)
- J2_DECK_B1 pad 6: Net-(ArduinoProMicroATmega32U4USB-C1-D14) -> Net-(SW_LOAD_B1-A)
Routing:
- net Net-(ArduinoProMicroATmega32U4USB-C1-~D6/A7): track 71.5 -> 56.2 mm
- net Net-(ArduinoProMicroATmega32U4USB-C1-D8/A8): track 74.1 -> 61.3 mm
- net Net-(ArduinoProMicroATmega32U4USB-C1-D4/A6): track 34.8 -> 22.2 mm, vias 1 -> 0
- net Net-(ArduinoProMicroATmega32U4USB-C1-D16): track 32.4 -> 40.2 mm, vias 0 -> 2
- net Net-(ArduinoProMicroATmega32U4USB-C1-VCC): track 88.0 -> 81.6 mm
- net Net-(ArduinoProMicroATmega32U4USB-C1-D2): track 18.9 -> 13.9 mm
- net Net-(ArduinoProMicroATmega32U4USB-C1-~D5): track 45.8 -> 42.6 mm, vias 1 -> 0
- net Net-(ArduinoProMicroATmega32U4USB-C1-~D9/A9): track 35.8 -> 38.2 mm, vias 1 -> 0
- net Net-(ArduinoProMicroATmega32U4USB-C1-D7): track 36.2 -> 34.6 mm
- net Net-(ArduinoProMicroATmega32U4USB-C1-~D3): track 17.9 -> 19.5 mm, vias 0 -> 1
- net Net-(ArduinoProMicroATmega32U4USB-C1-~D10/A10): track 64.5 -> 66.0 mm
- net GND: track 152.1 -> 151.0 mm, vias 0 -> 1
- net Net-(ArduinoProMicroATmega32U4USB-C1-D14): track 76.5 -> 77.6 mm
- net Net-(ROTARY_ENCODER_BTN1-SHIELD-PadSH1): track 18.0 -> 18.9 mm

Commit message: capacitors
Parts:
- renumbered R1_PLAY_A1 to R_PLAY_A1
Routing:
- net Net-(ArduinoProMicroATmega32U4USB-C1-D14): track 77.6 -> 52.4 mm, vias 1 -> 2
- net Net-(SW_LOAD_B1-A): track 0.00 -> 22.9 mm
- net Net-(SW_PLAY_A1-A): track 0.00 -> 19.6 mm
- net Net-(SW_LOAD_A1-A): track 0.00 -> 19.1 mm
- net Net-(SW_PLAY_B1-A): track 0.00 -> 14.2 mm
- net Net-(ArduinoProMicroATmega32U4USB-C1-D16): track 40.2 -> 51.3 mm, vias 2 -> 1
- net Net-(ArduinoProMicroATmega32U4USB-C1-~D9/A9): track 38.2 -> 28.5 mm, vias 0 -> 1
- net Net-(ArduinoProMicroATmega32U4USB-C1-~D10/A10): track 66.0 -> 56.4 mm, vias 1 -> 2
- net GND: track 151.0 -> 145.4 mm
- net Net-(ArduinoProMicroATmega32U4USB-C1-VCC): track 81.6 -> 77.3 mm
- net Net-(ROTARY_ENCODER_BTN1-SHIELD-PadSH1): track 18.9 -> 16.7 mm
- net Net-(ArduinoProMicroATmega32U4USB-C1-D18/A0): track 25.7 -> 27.1 mm
- net Net-(ArduinoProMicroATmega32U4USB-C1-~D6/A7): track 56.2 -> 54.8 mm
- net Net-(ArduinoProMicroATmega32U4USB-C1-D7): track 34.6 -> 33.3 mm
- net Net-(ArduinoProMicroATmega32U4USB-C1-~D3): track 19.5 -> 18.3 mm
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
Commit message: MULTIPCB
Parts:
- added C1: 100nF, Capacitor_SMD:C_0603_1608Metric, F.Cu at (143.5, 115.0)
- added C2: 10uF, Capacitor_SMD:C_0805_2012Metric, F.Cu at (148.8, 115.0)
- added REF**: MountingHole_3.2mm_M3_DIN965_Pad, MountingHole:MountingHole_3.2mm_M3_DIN965_Pad, F.Cu at (121.0, 150.5)
- added REF**: MountingHole_3.2mm_M3_DIN965_Pad, MountingHole:MountingHole_3.2mm_M3_DIN965_Pad, F.Cu at (180.0, 90.0)
- ArduinoProMicroATmega32U4USB-C1: value Sparkfun_Pro_Micro -> ArduinoProMicroATmega32U4USB-C1
- moved FADETUBE-LOGO 0.50 mm to (166.0, 150.5)
- moved ONDAAUDIO-LOGO 0.50 mm to (176.5, 150.5)
Routing:
- net Net-(ArduinoProMicroATmega32U4USB-C1-VCC): track 77.3 -> 97.7 mm, vias 1 -> 3
- net GND: track 145.4 -> 158.4 mm, vias 1 -> 2

Commit message: MVP PRIOR MANUFACTURING
Parts:
- ArduinoProMicroATmega32U4USBC-1: renamed from ArduinoProMicroATmega32U4USB-C1; value ArduinoProMicroATmega32U4USB-C1 -> ArduinoProMicroATmega32U4USBC-1
