File: FADETUBE_MIDI/FADETUBE_MIDI.kicad_pcb (KiCad board)
At the start: 2 copper layers, 70 x 70 mm, 15 parts, among them J1_DECK_A1 B8B-PH-K-S, J2_DECK_B1 B8B-PH-K-S

Commit message: BOMLIST INCLUDED
Parts:
- ArduinoProMicroATmega32U4USBC-1: value ArduinoProMicroATmega32U4USBC-1 -> SPARKFUN QWIIC PRO MICRO - USB-C
- C1: value 100nF -> 0.1 µF; footprint Capacitor_SMD:C_0603_1608Metric -> FADETUBE_LIBRARY:CAPC1608X90
- C2: value 10uF -> 10 µF; footprint Capacitor_SMD:C_0805_2012Metric -> FADETUBE_LIBRARY:CAPC2012X88N
- FADER1: value PTA4553-2215CIB103 -> PTA4553-2215CIB103 10k 45mm
- ROTARY_ENCODER_BTN1: value PEC11R-4220K-S0024 -> PEC11R-4220K-S0024 10k
- R_LOAD_A1, R_LOAD_B1, R_PLAY_A1, R_PLAY_B1: value 1k -> 470 Ohms; footprint Resistor_SMD:R_0603_1608Metric -> FADETUBE_LIBRARY:RESC1608X55
- moved C2 1.80 mm to (147.0, 115.0)
- moved C1 1.00 mm to (142.5, 115.0)
- moved R_LOAD_B1 0.18 mm to (153.5, 142.0)
- moved R_PLAY_A1 0.15 mm to (141.5, 141.8), turned to 90 degrees
- renumbered REF** to MH1, REF** to MH2
Connections:
- J1_DECK_A1 pad 2: Net-(SW_PLAY_A1-A) -> Net-(J1_DECK_A1-Pad2)
- J2_DECK_B1 pad 2: Net-(SW_PLAY_B1-A) -> Net-(J2_DECK_B1-Pad2)
- R_PLAY_A1 pad 1: Net-(ArduinoProMicroATmega32U4USBC-1-~D9/A9) -> Net-(J1_DECK_A1-Pad2)
- R_PLAY_A1 pad 2: Net-(SW_PLAY_A1-A) -> Net-(ArduinoProMicroATmega32U4USBC-1-~D9/A9)
- R_PLAY_B1 pad 1: Net-(ArduinoProMicroATmega32U4USBC-1-~D10/A10) -> Net-(J2_DECK_B1-Pad2)
- R_PLAY_B1 pad 2: Net-(SW_PLAY_B1-A) -> Net-(ArduinoProMicroATmega32U4USBC-1-~D10/A10)
Routing:
- net Net-(SW_PLAY_A1-A): track 19.6 -> 0.00 mm
- net Net-(J1_DECK_A1-Pad2): track 0.00 -> 19.4 mm
- net Net-(SW_PLAY_B1-A): track 14.2 -> 0.00 mm
- net GND: track 158.4 -> 172.3 mm, vias 2 -> 1
- net Net-(ArduinoProMicroATmega32U4USBC-1-VCC): track 97.7 -> 110.9 mm, vias 3 -> 1
- net Net-(J2_DECK_B1-Pad2): track 0.00 -> 9.34 mm
- net Net-(ArduinoProMicroATmega32U4USBC-1-~D10/A10): track 56.4 -> 64.5 mm, vias 2 -> 1
- net Net-(ArduinoProMicroATmega32U4USBC-1-D16): track 51.3 -> 45.3 mm
- net Net-(ArduinoProMicroATmega32U4USBC-1-D14): track 52.4 -> 57.8 mm
- net Net-(ArduinoProMicroATmega32U4USBC-1-D2): track 13.9 -> 18.0 mm, vias 0 -> 1
- net Net-(ArduinoProMicroATmega32U4USBC-1-~D6/A7): track 54.8 -> 58.3 mm
- net Net-(ArduinoProMicroATmega32U4USBC-1-~D9/A9): track 28.5 -> 26.1 mm
- net Net-(FADER1-SHIELD-PadSH1): track 68.2 -> 65.8 mm
- net Net-(ArduinoProMicroATmega32U4USBC-1-D8/A8): track 61.3 -> 59.1 mm
- net Net-(ROTARY_ENCODER_BTN1-SHIELD-PadSH1): track 16.7 -> 18.9 mm
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