File: FADETUBE_MIDI/FADETUBE_MIDI.kicad_pcb (KiCad board)
At the start: 2 copper layers, 180 x 70 mm, 28 parts, among them J1_DECK_A1 B8B-PH-K-S, J2_DECK_B1 B8B-PH-K-S

Commit message: updates
Parts:
- moved ArduinoProMicroATmega32U4USBC-1 2.00 mm to (-28.0, -0.50)
Routing:
- net Net-(ArduinoProMicroATmega32U4USBC-1-VCC): track 258.3 -> 279.3 mm, vias 2 -> 4
- net Net-(ArduinoProMicroATmega32U4USBC-1-D21/A3): track 91.9 -> 106.5 mm
- net Net-(ArduinoProMicroATmega32U4USBC-1-D14): track 52.1 -> 65.6 mm
- net Net-(ArduinoProMicroATmega32U4USBC-1-~D6/A7): track 54.6 -> 45.3 mm
- net Net-(ArduinoProMicroATmega32U4USBC-1-D15): track 88.6 -> 95.9 mm, vias 1 -> 2
- net Net-(ArduinoProMicroATmega32U4USBC-1-D20/A2): track 57.7 -> 62.7 mm, vias 0 -> 1
- net GND: track 320.8 -> 316.1 mm
- net Net-(ArduinoProMicroATmega32U4USBC-1-~D10/A10): track 45.7 -> 48.3 mm
- net Net-(FADER_CROSSFADER1-SHIELD-PadSH1): track 65.8 -> 68.2 mm
- net Net-(ArduinoProMicroATmega32U4USBC-1-D18/A0): track 26.3 -> 24.1 mm
- net Net-(ArduinoProMicroATmega32U4USBC-1-D0/RX): track 46.8 -> 44.8 mm
- net Net-(ArduinoProMicroATmega32U4USBC-1-~D5): track 39.8 -> 37.8 mm
- net Net-(ArduinoProMicroATmega32U4USBC-1-D7): track 32.0 -> 30.0 mm
- net Net-(ArduinoProMicroATmega32U4USBC-1-~D9/A9): track 21.8 -> 19.8 mm
- net Net-(J2_DECK_B1-Pad2): track 9.64 -> 11.4 mm
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
Commit message: UPDATES
Parts:
- C1, C2, R_LOAD_A1, R_LOAD_B1, R_PLAY_A1, R_PLAY_B1: moved to B.Cu
Other:
- board text added: "1 - PLAY A BTN"
- board text added: "1 - PLAY B BTN"
- board text added: "2 - PLAY A LED"
- board text added: "2 - PLAY B LED"
- board text added: "3 - PLAY A LED GND"
- board text added: "3 - PLAY B LED GND"
- board text added: "4 - PLAY A BTN GRND"
- board text added: "4 - PLAY B BTN GRND"
- board text added: "5 - LOAD A BTN"
- board text added: "5 - LOAD B BTN"
- board text added: "6 - LOAD A BTN LED"
- board text added: "6 - LOAD B BTN LED"
- board text added: "7 - LOAD A LED GND"
- board text added: "7 - LOAD B LED GND"
- board text added: "8 - LOAD A BTN GRND"
- board text added: "8 - LOAD B BTN GRND"
- board text added: "PLAY 1 BTN = PIN 8 - D5 PLAY 2 BTN = PIN 9 - D6 LOAD 1 BTN = 10 - D7 LOAD 2 BTN = 11 - D8 PLAY 1 BTN LED = 12 - D9 PLAY 2 BTN LED = 13 - D10 LOAD 1 BTN LED = 14 - D16 LOAD 2 BTN LED = 15 - D14"

Commit message: new updates
Parts:
- added JPH_DECK_A1: B4B-PH-K-S, FADETUBE_LIBRARY:JST_B4B-PH-K-S, B.Cu at (-27.7, 21.0)
- added JPH_DECK_A2: B4B-PH-K-S, FADETUBE_LIBRARY:JST_B4B-PH-K-S, B.Cu at (-17.1, 21.0)
- added JPH_DECK_B1: B4B-PH-K-S, FADETUBE_LIBRARY:JST_B4B-PH-K-S, B.Cu at (17.1, 21.0)
- added JPH_DECK_B2: B4B-PH-K-S, FADETUBE_LIBRARY:JST_B4B-PH-K-S, B.Cu at (27.7, 21.0)
- moved J2_DECK_B1 53.8 mm to (41.8, 69.7)
- moved J1_DECK_A1 43.2 mm to (-11.9, 62.3)
Connections:
- ROTARY_ENCODER_BTN1 pad 1: GND -> unconnected-(ROTARY_ENCODER_BTN1-Pad1)
- R_LOAD_A1 pad 1: Net-(J1_DECK_A1-Pad6) -> Net-(JPH_DECK_A2-Pad2)
- R_LOAD_B1 pad 1: Net-(J2_DECK_B1-Pad6) -> Net-(JPH_DECK_B2-Pad2)
- R_PLAY_A1 pad 1: Net-(J1_DECK_A1-Pad2) -> Net-(JPH_DECK_A1-Pad2)
- R_PLAY_B1 pad 1: Net-(J2_DECK_B1-Pad2) -> Net-(JPH_DECK_B1-Pad2)
Routing:
- net GND: track 316.1 -> 0.00 mm, vias 1 -> 0
- net Net-(ArduinoProMicroATmega32U4USBC-1-VCC): track 279.7 -> 0.00 mm, vias 4 -> 0
- net Net-(ArduinoProMicroATmega32U4USBC-1-D19/A1): track 118.4 -> 0.00 mm, vias 1 -> 0
- net Net-(ArduinoProMicroATmega32U4USBC-1-D21/A3): track 106.5 -> 0.00 mm, vias 1 -> 0
- net Net-(ArduinoProMicroATmega32U4USBC-1-D15): track 95.9 -> 0.00 mm, vias 2 -> 0
- net Net-(FADER_CROSSFADER1-SHIELD-PadSH1): track 68.2 -> 0.00 mm
- net Net-(FADER_TEMPO_B1-SHIELD-PadSH1): track 65.8 -> 0.00 mm
- net Net-(FADER_TEMPO_A1-SHIELD-PadSH1): track 65.8 -> 0.00 mm
- net Net-(ArduinoProMicroATmega32U4USBC-1-D14): track 65.6 -> 0.00 mm, vias 1 -> 0
- net Net-(ArduinoProMicroATmega32U4USBC-1-D20/A2): track 62.7 -> 0.00 mm, vias 1 -> 0
- net Net-(ArduinoProMicroATmega32U4USBC-1-D8/A8): track 54.9 -> 0.00 mm, vias 1 -> 0
- net Net-(ArduinoProMicroATmega32U4USBC-1-~D10/A10): track 48.3 -> 0.00 mm, vias 1 -> 0
- net Net-(ArduinoProMicroATmega32U4USBC-1-~D6/A7): track 45.3 -> 0.00 mm, vias 1 -> 0
- net Net-(ArduinoProMicroATmega32U4USBC-1-D16): track 45.1 -> 0.00 mm, vias 1 -> 0
- net Net-(ArduinoProMicroATmega32U4USBC-1-D0/RX): track 44.8 -> 0.00 mm
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Other:
- outline, holes or cut-outs redrawn
