File: FADETUBE_MIDI/FADETUBE_MIDI.kicad_sch (KiCad schematic)
At the start: 7 parts, among them J1 B8B-XH-A, J2 B8B-XH-A, J3 B8B-PH-K-S, J4 B8B-PH-K-S, U1 Sparkfun_Pro_Micro

Commit message: updates
Parts:
- removed J1, J2: B8B-XH-A, FADETUBE_LIBRARY:JST_B8B-XH-A, symbol FADETUBE_LIBRARY:B8B-XH-A
- added SW_LOAD_A1, SW_LOAD_B1, SW_PLAY_A1, SW_PLAY_B1: SW_Push_LED, symbol Switch:SW_Push_LED
- renumbered U1 to ArduinoProMicroATmega32U4USB-C1, R1 to FADER1, J3 to J1_DECK_A1, J4 to J2_DECK_B1, S1 to ROTARY_ENCODER_BTN1
Connections:
- net VCC is gone; now on an unnamed net: FADER1.3
- net GND: now also ArduinoProMicroATmega32U4USB-C1.3 (GND), ArduinoProMicroATmega32U4USB-C1.4 (GND), J1_DECK_A1.3, J1_DECK_A1.4, J1_DECK_A1.7, J1_DECK_A1.8, J2_DECK_B1.3, J2_DECK_B1.4, J2_DECK_B1.7, J2_DECK_B1.8, SW_LOAD_A1.1, SW_LOAD_A1.3 (K), SW_LOAD_B1.1, SW_LOAD_B1.3 (K), SW_PLAY_A1.1, SW_PLAY_A1.3 (K), SW_PLAY_B1.1, SW_PLAY_B1.3 (K)
- net at J1_DECK_A1.1: now also ArduinoProMicroATmega32U4USB-C1.8 (~D5), SW_PLAY_A1.2
- net at J1_DECK_A1.2: now also ArduinoProMicroATmega32U4USB-C1.12 (~D9/A9), SW_PLAY_A1.4 (A)
- net at J1_DECK_A1.5: now also ArduinoProMicroATmega32U4USB-C1.10 (D7), SW_LOAD_A1.2
- net at J1_DECK_A1.6: now also ArduinoProMicroATmega32U4USB-C1.14 (D16), SW_LOAD_A1.4 (A)
- net at J2_DECK_B1.1: now also ArduinoProMicroATmega32U4USB-C1.9 (~D6/A7), SW_PLAY_B1.2
- net at J2_DECK_B1.2: now also ArduinoProMicroATmega32U4USB-C1.13 (~D10/A10), SW_PLAY_B1.4 (A)
- net at J2_DECK_B1.5: now also ArduinoProMicroATmega32U4USB-C1.11 (D8/A8), SW_LOAD_B1.2
- net at J2_DECK_B1.6: now also ArduinoProMicroATmega32U4USB-C1.15 (D14), SW_LOAD_B1.4 (A)
- net at ROTARY_ENCODER_BTN1.2: now also ArduinoProMicroATmega32U4USB-C1.7 (D4/A6); no longer ArduinoProMicroATmega32U4USB-C1.4 (GND)
Other:
- moved on the sheet: FADER1, J1_DECK_A1, J2_DECK_B1, ROTARY_ENCODER_BTN1

Commit message: test smd
Parts:
- added R1_PLAY_A, R_LOAD_A, R_LOAD_B, R_PLAY_B: 1k, Resistor_SMD:R_0603_1608Metric, symbol Device:R_US
Connections:
- net at J2_DECK_B1.6, SW_LOAD_B1.4 (A): now also R_LOAD_B.1; no longer ArduinoProMicroATmega32U4USB-C1.15 (D14)
- net at J1_DECK_A1.2, SW_PLAY_A1.4 (A): now also R1_PLAY_A.2; no longer ArduinoProMicroATmega32U4USB-C1.12 (~D9/A9)
- net at J1_DECK_A1.6, SW_LOAD_A1.4 (A): now also R_LOAD_A.1; no longer ArduinoProMicroATmega32U4USB-C1.14 (D16)
- net at J2_DECK_B1.2, SW_PLAY_B1.4 (A): now also R_PLAY_B.2; no longer ArduinoProMicroATmega32U4USB-C1.13 (~D10/A10)
- new net: ArduinoProMicroATmega32U4USB-C1.13 (~D10/A10), R_PLAY_B.1
- new net: ArduinoProMicroATmega32U4USB-C1.15 (D14), R_LOAD_B.2
- new net: ArduinoProMicroATmega32U4USB-C1.14 (D16), R_LOAD_A.2
- new net: ArduinoProMicroATmega32U4USB-C1.12 (~D9/A9), R1_PLAY_A.1
Other:
- moved on the sheet: ArduinoProMicroATmega32U4USB-C1, FADER1, J1_DECK_A1, J2_DECK_B1, ROTARY_ENCODER_BTN1, SW_LOAD_A1, SW_LOAD_B1, SW_PLAY_A1, SW_PLAY_B1

Commit message: capacitors
Parts:
- ArduinoProMicroATmega32U4USB-C1: value Sparkfun_Pro_Micro -> ArduinoProMicroATmega32U4USB-C1
- renumbered R_LOAD_A to R_LOAD_A1, R_LOAD_B to R_LOAD_B1, R1_PLAY_A to R_PLAY_A1, R_PLAY_B to R_PLAY_B1
Changed lines of the file:
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@@
 		(on_board yes)
 		(dnp no)
-		(property "Reference" "R_PLAY_B"
+		(property "Reference" "R_PLAY_B1"
 			(at 107.95 116.8399 0)
 			(effects
@@
 			(project "FADETUBE_MIDI"
 				(path "/51aff578-2ad6-4f14-ac60-9cc95c2688c8"
-					(reference "R_PLAY_B")
+					(reference "R_PLAY_B1")
 					(unit 1)
 				)
@@
 		(on_board yes)
 		(dnp no)
-		(property "Reference" "R_LOAD_B"
+		(property "Reference" "R_LOAD_B1"
 			(at 115.57 132.08 90)
 			(effects
@@
 			(project "FADETUBE_MIDI"
 				(path "/51aff578-2ad6-4f14-ac60-9cc95c2688c8"
-					(reference "R_LOAD_B")
+					(reference "R_LOAD_B1")
 					(unit 1)
 				)
@@
 		(on_board yes)
 		(dnp no)
-		(property "Reference" "R_LOAD_A"
+		(property "Reference" "R_LOAD_A1"
 			(at 113.03 90.678 90)
 			(effects
@@
 			(project "FADETUBE_MIDI"
 				(path "/51aff578-2ad6-4f14-ac60-9cc95c2688c8"
-					(reference "R_LOAD_A")
+					(reference "R_LOAD_A1")
 					(unit 1)
 				)
@@
 		(on_board yes)
 		(dnp no)
-		(property "Reference" "R1_PLAY_A"
+		(property "Reference" "R_PLAY_A1"
 			(at 106.68 72.3899 0)
 			(effects
@@
 			(project ""
 				(path "/51aff578-2ad6-4f14-ac60-9cc95c2688c8"
-					(reference "R1_PLAY_A")
+					(reference "R_PLAY_A1")
 					(unit 1)
 				)
@@
 			)
 		)
-		(property "Value" "Sparkfun_Pro_Micro"
+		(property "Value" "ArduinoProMicroATmega32U4USB-C1"
 			(at 102.87 31.75 0)
 			(effects

Commit message: MULTIPCB
Parts:
- added C1: 100nF, Capacitor_SMD:C_0603_1608Metric, symbol Device:C_US
- added C2: 10uF, Capacitor_SMD:C_0805_2012Metric, symbol Device:C_US
Connections:
- net GND: now also C1.1, C2.1
- net at ArduinoProMicroATmega32U4USB-C1.21 (VCC), FADER1.3: now also C1.2, C2.2
Changed lines of the file:
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@@
+	)
+	(junction
+		(at 133.35 44.45)
+		(diameter 0)
+		(color 0 0 0 0)
 	)
 	(junction
@@
 	)
 	(junction
+		(at 133.35 25.4)
+		(diameter 0)
+		(color 0 0 0 0)
+	)
+	(junction
+		(at 154.94 25.4)
+		(diameter 0)
+		(color 0 0 0 0)
+	)
+	(junction
 		(at 83.82 124.46)
 		(diameter 0)
@@
 	)
 	(junction
+		(at 154.94 44.45)
+		(diameter 0)
+		(color 0 0 0 0)
+	)
+	(junction
 		(at 83.82 127)
 		(diameter 0)
@@
 	(wire
 		(pts
+			(xy 133.35 39.37) (xy 133.35 44.45)
+		)
+		(stroke
+			(width 0)
+			(type default)
+		)
+	)
+	(wire
+		(pts
 			(xy 34.29 90.17) (xy 35.56 90.17)
 		)
@@
 	(wire
 		(pts
+			(xy 154.94 25.4) (xy 154.94 31.75)
+		)
+		(stroke
+			(width 0)
+			(type default)
+		)
+	)
+	(wire
+		(pts
 			(xy 45.72 92.71) (xy 83.82 92.71)
 		)
@@
 	(wire
 		(pts
+			(xy 133.35 25.4) (xy 154.94 25.4)
+		)
+		(stroke
+			(width 0)
+			(type default)
+		)
+	)
+	(wire
+		(pts
 			(xy 83.82 87.63) (xy 49.53 87.63)
 		)
@@
 	(wire
 		(pts
+			(xy 154.94 44.45) (xy 171.45 44.45)
+		)
+		(stroke
+			(width 0)
+			(type default)
+		)
+	)
+	(wire
+		(pts
 			(xy 135.89 97.79) (xy 135.89 127)
 		)
@@
 	(wire
 		(pts
+			(xy 154.94 39.37) (xy 154.94 44.45)
+		)
+		(stroke
+			(width 0)
+			(type default)
+		)
+	)
+	(wire
+		(pts
 			(xy 83.82 95.25) (xy 135.89 95.25)
 		)
@@
 	(wire
 		(pts
+			(xy 133.35 44.45) (xy 154.94 44.45)
+		)
+		(stroke
+			(width 0)
+			(type default)
+		)
+	)
+	(wire
+		(pts
 			(xy 85.09 33.02) (xy 85.09 41.91)
 		)
@@
 	(wire
 		(pts
-			(xy 77.47 25.4) (xy 179.07 25.4)
+			(xy 77.47 25.4) (xy 133.35 25.4)
 		)
 		(stroke
@@
 	(wire
 		(pts
+			(xy 133.35 25.4) (xy 133.35 31.75)
+		)
+		(stroke
+			(width 0)
+			(type default)
+		)
+	)
+	(wire
+		(pts
 			(xy 77.47 59.69) (xy 77.47 90.17)
 		)
@@
 	(wire
 		(pts
-			(xy 118.11 44.45) (xy 171.45 44.45)
+			(xy 118.11 44.45) (xy 133.35 44.45)
 		)
 		(stroke
@@
 		(pts
 			(xy 74.93 54.61) (xy 87.63 54.61)
+		)
+		(stroke
+			(width 0)
+			(type default)
+		)
+	)
+	(wire
+		(pts
+			(xy 154.94 25.4) (xy 179.07 25.4)
 		)
 		(stroke
@@
 	)
 	(symbol
+		(lib_id "Device:C_US")
+		(at 133.35 35.56 0)
+		(unit 1)
+		(exclude_from_sim no)
+		(in_bom yes)
+		(on_board yes)
+		(dnp no)
+		(property "Reference" "C1"
+			(at 137.16 34.5439 0)
+			(effects
+				(font
+					(size 1.27 1.27)
+				)
+				(justify left)
+			)
+		)
+		(property "Value" "100nF"
+			(at 137.16 37.0839 0)
+			(effects
+				(font
+					(size 1.27 1.27)
+				)
+				(justify left)
+			)
+		)
+		(property "Footprint" "Capacitor_SMD:C_0603_1608Metric"
+			(at 133.35 35.56 0)
+			(effects
+				(font
+					(size 1.27 1.27)
+				)
+				(hide yes)
+			)
+		)
+		(property "Datasheet" ""
+			(at 133.35 35.56 0)
+			(effects
+				(font
+					(size 1.27 1.27)
+				)
+				(hide yes)
+			)
+		)
+		(property "Description" "capacitor, US symbol"
+			(at 133.35 35.56 0)
+			(effects
+				(font
+					(size 1.27 1.27)
+				)
+				(hide yes)
+			)
+		)
+		(pin "1"
+		)
+		(pin "2"
+		)
+		(instances
+			(project ""
+				(path "/51aff578-2ad6-4f14-ac60-9cc95c2688c8"
+					(reference "C1")
+					(unit 1)
+				)
+			)
+		)
+	)
+	(symbol
 		(lib_id "Device:R_US")
 		(at 113.03 134.62 90)
@@
 					(unit 1)
 				)
+			)
+		)
+	)
+	(symbol
+		(lib_id "Device:C_US")
+		(at 154.94 35.56 0)
+		(unit 1)
+		(exclude_from_sim no)
+		(in_bom yes)
+		(on_board yes)
+		(dnp no)
+		(fields_autoplaced yes)
+		(property "Reference" "C2"
+			(at 158.75 34.5439 0)
+			(effects
+				(font
+					(size 1.27 1.27)
+				)
+				(justify left)
+			)
+		)
+		(property "Value" "10uF"
+			(at 158.75 37.0839 0)
+			(effects
+				(font
+					(size 1.27 1.27)
+				)
+				(justify left)
+			)
+		)
+		(property "Footprint" "Capacitor_SMD:C_0805_2012Metric"
+			(at 154.94 35.56 0)
+			(effects
+				(font
+					(size 1.27 1.27)
+				)
+				(hide yes)
+			)
+		)
+		(property "Datasheet" ""
+			(at 154.94 35.56 0)
+			(effects
+				(font
+					(size 1.27 1.27)
+				)
+				(hide yes)
+			)
+		)
+		(property "Description" "capacitor, US symbol"
+			(at 154.94 35.56 0)
+			(effects
+				(font
+					(size 1.27 1.27)
+				)
+				(hide yes)
+			)
+		)
+		(pin "1"
+		)
+		(pin "2"
+		)
+		(instances
+			(project "FADETUBE_MIDI"
+				(path "/51aff578-2ad6-4f14-ac60-9cc95c2688c8"
+					(reference "C2")
+					(unit 1)
+				)

Commit message: MVP PRIOR MANUFACTURING
Parts:
- ArduinoProMicroATmega32U4USBC-1: renamed from ArduinoProMicroATmega32U4USB-C1; value ArduinoProMicroATmega32U4USB-C1 -> ArduinoProMicroATmega32U4USBC-1
Changed lines of the file:
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@@
 		(dnp no)
 		(fields_autoplaced yes)
-		(property "Reference" "ArduinoProMicroATmega32U4USB-C1"
+		(property "Reference" "ArduinoProMicroATmega32U4USBC-1"
 			(at 102.87 29.21 0)
 			(effects
@@
 			)
 		)
-		(property "Value" "ArduinoProMicroATmega32U4USB-C1"
+		(property "Value" "ArduinoProMicroATmega32U4USBC-1"
 			(at 102.87 31.75 0)
 			(effects
@@
 			)
 		)
-		(property "Datasheet" "https://www.sparkfun.com/products/12640"
+		(property "Datasheet" "https://cdn.sparkfun.com/assets/learn_tutorials/1/1/1/4/QwiicProMicroUSB-C.pdf"
 			(at 105.41 78.74 0)
 			(effects
@@
 			)
 		)
-		(property "Description" "Sparkfun Pro Micro"
+		(property "Description" "SPARKFUN QWIIC PRO MICRO - USB-C"
 			(at 102.87 52.07 0)
 			(effects
@@
 			(project ""
 				(path "/51aff578-2ad6-4f14-ac60-9cc95c2688c8"
-					(reference "ArduinoProMicroATmega32U4USB-C1")
+					(reference "ArduinoProMicroATmega32U4USBC-1")
 					(unit 1)
 				)
