File: FADETUBE_MIDI/FADETUBE_MIDI.kicad_sch (KiCad schematic)
At the start: 15 parts, among them J1_DECK_A1 B8B-PH-K-S, J2_DECK_B1 B8B-PH-K-S

Commit message: BOMLIST INCLUDED
Parts:
- removed C1: 100nF, Capacitor_SMD:C_0603_1608Metric, symbol Device:C_US
- removed C2: 10uF, Capacitor_SMD:C_0805_2012Metric, symbol Device:C_US
- removed R_LOAD_A1, R_LOAD_B1, R_PLAY_A1, R_PLAY_B1: 1k, Resistor_SMD:R_0603_1608Metric, symbol Device:R_US
- added C1: 0.1 µF, FADETUBE_LIBRARY:CAPC1608X90, symbol FADETUBE_LIBRARY:C0603C104K4RACTU
- added C2: 10 µF, FADETUBE_LIBRARY:CAPC2012X88N, symbol FADETUBE_LIBRARY:C0805C106K8PACTU
- added R_LOAD_A1, R_LOAD_B1, R_PLAY_A1, R_PLAY_B1: 470 Ohms, FADETUBE_LIBRARY:RESC1608X55, symbol FADETUBE_LIBRARY:RC0603FR-07470RL
- ArduinoProMicroATmega32U4USBC-1, J1_DECK_A1, J2_DECK_B1: SUPPLIER digikey -> DIGIKEY
- FADER1, ROTARY_ENCODER_BTN1: MANUFACTURER Bourns -> BOURNS; SUPPLIER digikey -> DIGIKEY
Connections:
- net GND: now also C1.1, C2.1
- net at ArduinoProMicroATmega32U4USBC-1.13 (~D10/A10): now also R_PLAY_B1.2
- net at J2_DECK_B1.2, SW_PLAY_B1.4 (A): now also R_PLAY_B1.1
- net at J2_DECK_B1.6, SW_LOAD_B1.4 (A): now also R_LOAD_B1.1
- net at J1_DECK_A1.2, SW_PLAY_A1.4 (A): now also R_PLAY_A1.1
- net at J1_DECK_A1.6, SW_LOAD_A1.4 (A): now also R_LOAD_A1.1
- net at ArduinoProMicroATmega32U4USBC-1.21 (VCC), FADER1.3: now also C1.2, C2.2
- net at ArduinoProMicroATmega32U4USBC-1.15 (D14): now also R_LOAD_B1.2
- net at ArduinoProMicroATmega32U4USBC-1.14 (D16): now also R_LOAD_A1.2
- net at ArduinoProMicroATmega32U4USBC-1.12 (~D9/A9): now also R_PLAY_A1.2
