File: bk/_autosave-FADETUBE_MIDI.kicad_sch (KiCad schematic)
At the start: 21 parts, among them J1_DECK_A1 B8B-PH-K-S, J2_DECK_B1 B8B-PH-K-S

Commit message: ADVANCDED VERTION
Connections:
- net GND: now also C2.2; no longer C2.1
- net at ArduinoProMicroATmega32U4USBC-1.21 (VCC), C1.2, FADER_CROSSFADER1.3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: now also C2.1; no longer C2.2
Other:
- moved on the sheet: C2
Changed lines of the file:
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@@
 	(wire
 		(pts
-			(xy 153.67 74.93) (xy 153.67 80.01)
-		)
-		(stroke
-			(width 0)
-			(type default)
-		)
-	)
-	(wire
-		(pts
 			(xy 82.55 130.81) (xy 134.62 130.81)
 		)
@@
 	(wire
 		(pts
+			(xy 153.67 74.93) (xy 153.67 80.01)
+		)
+		(stroke
+			(width 0)
+			(type default)
+		)
+	)
+	(wire
+		(pts
 			(xy 245.11 92.71) (xy 250.19 92.71)
 		)
@@
 	(symbol
 		(lib_id "FADETUBE_LIBRARY:C0805C106K8PACTU")
-		(at 153.67 72.39 90)
+		(at 153.67 69.85 270)
 		(unit 1)
 		(exclude_from_sim no)
@@
 					(size 1.27 1.27)
 				)
-				(justify right)
+				(justify left)
 			)
 		)
@@
 					(size 1.27 1.27)
 				)
-				(justify right)
+				(justify left)
 			)
 		)
 		(property "Footprint" "Capacitor_THT:CP_Radial_D5.0mm_P2.00mm"
-			(at 153.67 72.39 0)
+			(at 153.67 69.85 0)
 			(effects
 				(font
@@
 		)
 		(property "Datasheet" "https://yageogroup.com/content/datasheet/asset/file/KEM_C1006_X5R_SMD"
-			(at 153.67 72.39 0)
+			(at 153.67 69.85 0)
 			(effects
 				(font
@@
 		)
 		(property "Description" "10 µF C0805C106K8PACTU"
-			(at 153.67 72.39 0)
+			(at 153.67 69.85 0)
 			(effects
 				(font
@@
 		)
 		(property "MF" "KEMET"
-			(at 153.67 72.39 0)
+			(at 153.67 69.85 0)
 			(effects
 				(font
@@
 		)
 		(property "Description_1" "0805 C 10uF Ceramic Multilayer Capacitor, 10 V, +85degC, X5R Dielectric, +/-10% | KEMET C0805C106K8PACTU"
-			(at 153.67 72.39 0)
+			(at 153.67 69.85 0)
 			(effects
 				(font
@@
 		)
 		(property "Package" "0805 Kemet"
-			(at 153.67 72.39 0)
+			(at 153.67 69.85 0)
 			(effects
 				(font
@@
 		)
 		(property "Price" "None"
-			(at 153.67 72.39 0)
+			(at 153.67 69.85 0)
 			(effects
 				(font
@@
 		)
 		(property "SnapEDA_Link" "https://www.snapeda.com/parts/C0805C106K8PACTU/Kemet/view-part/?ref=snap"
-			(at 153.67 72.39 0)
+			(at 153.67 69.85 0)
 			(effects
 				(font
@@
 		)
 		(property "MP" "C0805C106K8PACTU"
-			(at 153.67 72.39 0)
+			(at 153.67 69.85 0)
 			(effects
 				(font
@@
 		)
 		(property "Availability" "In Stock"
-			(at 153.67 72.39 0)
+			(at 153.67 69.85 0)
 			(effects
 				(font
@@
 		)
 		(property "Check_prices" "https://www.snapeda.com/parts/C0805C106K8PACTU/Kemet/view-part/?ref=eda"
-			(at 153.67 72.39 0)
+			(at 153.67 69.85 0)
 			(effects
 				(font
@@
 		)
 		(property "MANUFACTURER" "KEMET"
-			(at 153.67 72.39 90)
+			(at 153.67 69.85 90)
 			(effects
 				(font
@@
 		)
 		(property "MANUFACTURER PART NUMBER" "C0805C106K8PACTU"
-			(at 153.67 72.39 90)
+			(at 153.67 69.85 90)
 			(effects
 				(font
@@
 		)
 		(property "PURCHASE-URL" "https://www.digikey.com/en/products/detail/kemet/C0805C106K8PACTU/1090830?utm_campaign=buynow&utm_medium=aggregator&utm_source=snapeda"
-			(at 153.67 72.39 90)
+			(at 153.67 69.85 90)
 			(effects
 				(font
@@
 		)
 		(property "SUPPLIER" "DIGIKEY"
-			(at 153.67 72.39 90)
+			(at 153.67 69.85 90)
 			(effects
 				(font
@@
 		)
 		(property "SUPPLIER PART NUMBER" "399-C0805C106K8PACTUDKR-ND"
-			(at 153.67 72.39 90)
+			(at 153.67 69.85 90)
 			(effects
 				(font
